Commit message: almost done but map frame id issue

File: urdf/base.xacro (robot description, xacro)
@@ -6,5 +6,5 @@
     <xacro:property name="wheel_radius" value="0.053" />
     <xacro:property name="wheel_length" value="0.05" />
-    <!-- <link name="${robot_prefix}base_footprint" /> -->
+    <link name="${robot_prefix}base_footprint" />
     <link name="${robot_prefix}base_link">
         <visual>
@@ -23,9 +23,9 @@
         </collision>
     </link>
-    <!-- <joint name="${robot_prefix}base_footprint_joint" type="fixed">
+    <joint name="${robot_prefix}base_footprint_joint" type="fixed">
+        <child link="${robot_prefix}base_link" />
         <parent link="${robot_prefix}base_footprint" />
-        <child link="${robot_prefix}base_link" />
         <origin xyz="0 0 0.071" rpy="0 0 0"/>
-    </joint> -->
+    </joint>
     <xacro:macro name="wheel_link" params="prefix">
         <link name="${robot_prefix}${prefix}_wheel_link">
@@ -389,6 +389,6 @@
         </plugin>
     </gazebo>
-    <!-- Individual sensors plugin with unique scene name per robot -->
-    <!-- <gazebo>
+    <!-- Individual sensors plugin with unique scene name per robot
+    <gazebo>
         <plugin filename="gz-sim-sensors-system"
                 name="gz::sim::systems::Sensors">

Commit message: improvements in scan_merger_v2

File: urdf/base.xacro (robot description, xacro)
@@ -24,7 +24,7 @@
     </link>
     <joint name="${robot_prefix}base_footprint_joint" type="fixed">
-        <child link="${robot_prefix}base_link" />
-        <parent link="${robot_prefix}base_footprint" />
-        <origin xyz="0 0 0.071" rpy="0 0 0"/>
+        <parent link="${robot_prefix}base_link" />
+        <child link="${robot_prefix}base_footprint" />
+        <origin xyz="0 0 -0.071" rpy="0 0 0"/>
     </joint>
     <xacro:macro name="wheel_link" params="prefix">
@@ -60,5 +60,5 @@
         <axis xyz="0 1 0" />
     </joint>
-    <link name="${robot_prefix}gpu_lidar_right">
+    <link name="${robot_name_prefix}${robot_prefix}base_link/gpu_lidar_right">
         <visual>
             <geometry>
@@ -77,8 +77,8 @@
     <joint name="${robot_prefix}lidar_right_base_joint" type="fixed">
         <parent link="${robot_prefix}base_link" />
-        <child link="${robot_prefix}gpu_lidar_right" />
+        <child link="${robot_name_prefix}${robot_prefix}base_link/gpu_lidar_right" />
         <origin xyz="0.115 -0.16789 0.12" rpy="0 0 0"/>
     </joint>
-    <link name="${robot_prefix}gpu_lidar_left">
+    <link name="${robot_name_prefix}${robot_prefix}base_link/gpu_lidar_left">
         <visual>
             <geometry>
@@ -97,5 +97,5 @@
     <joint name="${robot_prefix}lidar_left_base_joint" type="fixed">
         <parent link="${robot_prefix}base_link" />
-        <child link="${robot_prefix}gpu_lidar_left" />
+        <child link="${robot_name_prefix}${robot_prefix}base_link/gpu_lidar_left" />
         <origin xyz="-0.115 0.16789 0.12" rpy="0 0 3.14"/>
     </joint>
@@ -313,8 +313,8 @@
         </sensor>
     </gazebo>
-    <gazebo reference="${robot_prefix}gpu_lidar_right">
+    <gazebo reference="${robot_name_prefix}${robot_prefix}base_link/gpu_lidar_right">
         <material>Gazebo/Black</material>
         <sensor name='gpu_lidar_right' type='gpu_lidar'>
-            <pose relative_to='${robot_prefix}gpu_lidar_right'>0 0 0 0 0 0</pose>
+            <pose relative_to='${robot_name_prefix}${robot_prefix}base_link/gpu_lidar_right'>0 0 0 0 0 0</pose>
             <topic>${namespace}/lidar1</topic>
             <update_rate>10</update_rate>
@@ -344,8 +344,8 @@
         </sensor>
     </gazebo>
-    <gazebo reference="${robot_prefix}gpu_lidar_left">
+    <gazebo reference="${robot_name_prefix}${robot_prefix}base_link/gpu_lidar_left">
         <material>Gazebo/Black</material>
         <sensor name='gpu_lidar_left' type='gpu_lidar'>
-            <pose relative_to='${robot_prefix}gpu_lidar_left'>0 0 0 0 0 0</pose>
+            <pose relative_to='${robot_name_prefix}${robot_prefix}base_link/gpu_lidar_left'>0 0 0 0 0 0</pose>
             <topic>${namespace}/lidar2</topic>
             <update_rate>10</update_rate>

File: urdf/dose_car.urdf.xacro (robot description, xacro)
@@ -9,4 +9,5 @@
     <!-- Keep robot_prefix empty - let robot_state_publisher handle frame prefixing -->
     <xacro:property name="robot_prefix" value="${namespace}/"/>
+    <xacro:property name="robot_name_prefix" value="${robot_name}/"/>
     <xacro:include filename="properties.xacro" />
     <xacro:include filename="base.xacro" />
